File: hardware/dac.sch (KiCad schematic (older format))
At the start: 39 parts

Commit message: more work on tdr schematic
Parts:
- U?: symbol symbols:AD9740ACPZ -> tdr-rescue:AD9740ACPZ-symbols
- U?: symbol synth_lib:ADA4817-1 -> tdr-rescue:ADA4817-1-synth_lib
Changed lines of the file:
@@
 $Descr A4 11693 8268
 encoding utf-8
-Sheet 6 9
+Sheet 7 9
 Title ""
 Date ""
@@
 $EndComp
 $Comp
-L symbols:AD9740ACPZ U?
+L tdr-rescue:AD9740ACPZ-symbols U?
 U 1 1 5BC36C50
 P 3800 1200
 AR Path="/5BC3F67C/5BC36C50" Ref="U?"  Part="1"
 AR Path="/5BC349EC/5BC36C50" Ref="U?"  Part="1"
+AR Path="/5BC36C50" Ref="U?"  Part="1"
 F 0 "U?" H 5043 1587 60  0000 C CNN
 F 1 "AD9740ACPZ" H 5043 1481 60  0000 C CNN
@@
 	7150 2650 7150 2500
 $Comp
-L synth_lib:ADA4817-1 U?
+L tdr-rescue:ADA4817-1-synth_lib U?
 U 1 1 5BC6297A
 P 8850 1750

Commit message: work on tdr schematic..
Parts:
- U?: symbol tdr-rescue:AD9740ACPZ-symbols -> tdr-rescue:AD9740ACPZ-symbols-tdr-rescue
- U?: symbol tdr-rescue:ADA4817-1-synth_lib -> tdr-rescue:ADA4817-1-synth_lib-tdr-rescue
Other:
- note added: "TODO: replace with 3V3 OP AMP"
Changed lines of the file:
@@
 $EndComp
 $Comp
-L tdr-rescue:AD9740ACPZ-symbols U?
+L tdr-rescue:AD9740ACPZ-symbols-tdr-rescue U?
 U 1 1 5BC36C50
 P 3800 1200
@@
 	7150 2650 7150 2500
 $Comp
-L tdr-rescue:ADA4817-1-synth_lib U?
+L tdr-rescue:ADA4817-1-synth_lib-tdr-rescue U?
 U 1 1 5BC6297A
 P 8850 1750
@@
 Wire Wire Line
 	8300 950  8300 1050
+Text Notes 8050 750  0    50   ~ 0
+TODO: replace with 3V3 OP AMP
 $EndSCHEMATC
