File: hardware/conn_power.sch (KiCad schematic (older format))
At the start: 63 parts, among them J201 Conn_02x01, J202 Conn_Coaxial, J203 Conn_Coaxial, J204 Conn_Coaxial, J205 Conn_Coaxial, J207 Conn_Coaxial, J208 Conn_Coaxial, J209 Conn_Coaxial, J210 Barrel_Jack_Switch, Q201 SI2369DS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

Commit message: more layout.. 28 unrouted nets to go
Parts:
- J208, J209: footprint vna_footprints:732511150_sma_thin -> vna_footprints:732511150_sma_thin_twopin
Changed lines of the file:
@@
 F 0 "J208" H 15149 6426 50  0000 L CNN
 F 1 "Conn_Coaxial" H 15149 6335 50  0000 L CNN
-F 2 "vna_footprints:732511150_sma_thin" H 15050 6450 50  0001 C CNN
+F 2 "vna_footprints:732511150_sma_thin_twopin" H 15050 6450 50  0001 C CNN
 F 3 " ~" H 15050 6450 50  0001 C CNN
 	1    15050 6450
@@
 F 0 "J209" H 15149 7276 50  0000 L CNN
 F 1 "Conn_Coaxial" H 15149 7185 50  0000 L CNN
-F 2 "vna_footprints:732511150_sma_thin" H 15050 7300 50  0001 C CNN
+F 2 "vna_footprints:732511150_sma_thin_twopin" H 15050 7300 50  0001 C CNN
 F 3 " ~" H 15050 7300 50  0001 C CNN
 	1    15050 7300

Commit message: schematic cleanup, BOM consolidation
Parts:
- C201, C202, C205, C212, C213: value 2.2 uF -> 4.7 uF
- C211: value 2.2 uF -> 10 uF
- R203, R205: value TBD -> DNI
- R216, R219: value TBD -> 1M
- R217, R218: value TBD -> 332k
- R220, R221: value R_Small -> JMP
- U201: value LD39100 -> LD39100PU33R
Other:
- note added: "R1"
- note added: "R2"
- note added: "R3"
- note added: "R4"
- note added: "VOUT+ = 1.2 V × (R1 + R2) / R2\nVOUT- = –1.22 V × (R3 + R4) / R4\nR must be no less than 50k"
Changed lines of the file:
@@
 P 4850 2650
 F 0 "U201" H 4850 3037 60  0000 C CNN
-F 1 "LD39100" H 4850 2931 60  0000 C CNN
+F 1 "LD39100PU33R" H 4850 2931 60  0000 C CNN
 F 2 "Housings_DFN_QFN:DFN-6-1EP_3x3mm_Pitch0.95mm" H 4850 2650 60  0001 C CNN
 F 3 "" H 4850 2650 60  0001 C CNN
@@
 P 5000 4650
 F 0 "C211" H 5092 4696 50  0000 L CNN
-F 1 "2.2 uF" H 5092 4605 50  0000 L CNN
+F 1 "10 uF" H 5092 4605 50  0000 L CNN
 F 2 "Capacitors_SMD:C_0603" H 5000 4650 50  0001 C CNN
 F 3 "~" H 5000 4650 50  0001 C CNN
@@
 P 5000 5250
 F 0 "R216" H 5059 5296 50  0000 L CNN
-F 1 "TBD" H 5059 5205 50  0000 L CNN
+F 1 "1M" H 5059 5205 50  0000 L CNN
 F 2 "Resistors_SMD:R_0402" H 5000 5250 50  0001 C CNN
 F 3 "~" H 5000 5250 50  0001 C CNN
@@
 P 5000 5550
 F 0 "R217" H 5059 5596 50  0000 L CNN
-F 1 "TBD" H 5059 5505 50  0000 L CNN
+F 1 "332k" H 5059 5505 50  0000 L CNN
 F 2 "Resistors_SMD:R_0402" H 5000 5550 50  0001 C CNN
 F 3 "~" H 5000 5550 50  0001 C CNN
@@
 P 5000 5850
 F 0 "R218" H 5059 5896 50  0000 L CNN
-F 1 "TBD" H 5059 5805 50  0000 L CNN
+F 1 "332k" H 5059 5805 50  0000 L CNN
 F 2 "Resistors_SMD:R_0402" H 5000 5850 50  0001 C CNN
 F 3 "~" H 5000 5850 50  0001 C CNN
@@
 P 5000 6150
 F 0 "R219" H 5059 6196 50  0000 L CNN
-F 1 "TBD" H 5059 6105 50  0000 L CNN
+F 1 "1M" H 5059 6105 50  0000 L CNN
 F 2 "Resistors_SMD:R_0402" H 5000 6150 50  0001 C CNN
 F 3 "~" H 5000 6150 50  0001 C CNN
@@
 P 5550 5350
 F 0 "C212" H 5642 5396 50  0000 L CNN
-F 1 "2.2 uF" H 5642 5305 50  0000 L CNN
+F 1 "4.7 uF" H 5642 5305 50  0000 L CNN
 F 2 "Capacitors_SMD:C_0603" H 5550 5350 50  0001 C CNN
 F 3 "~" H 5550 5350 50  0001 C CNN
@@
 P 5550 5950
 F 0 "C213" H 5642 5996 50  0000 L CNN
-F 1 "2.2 uF" H 5642 5905 50  0000 L CNN
+F 1 "4.7 uF" H 5642 5905 50  0000 L CNN
 F 2 "Capacitors_SMD:C_0603" H 5550 5950 50  0001 C CNN
 F 3 "~" H 5550 5950 50  0001 C CNN
@@
 P 6050 6300
 F 0 "R221" V 6246 6300 50  0000 C CNN
-F 1 "R_Small" V 6155 6300 50  0000 C CNN
+F 1 "JMP" V 6155 6300 50  0000 C CNN
 F 2 "Resistors_SMD:R_0402" H 6050 6300 50  0001 C CNN
 F 3 "~" H 6050 6300 50  0001 C CNN
@@
 P 6000 5100
 F 0 "R220" V 6196 5100 50  0000 C CNN
-F 1 "R_Small" V 6105 5100 50  0000 C CNN
+F 1 "JMP" V 6105 5100 50  0000 C CNN
 F 2 "Resistors_SMD:R_0402" H 6000 5100 50  0001 C CNN
 F 3 "~" H 6000 5100 50  0001 C CNN
@@
 P 3000 4750
 F 0 "C205" H 2908 4704 50  0000 R CNN
-F 1 "2.2 uF" H 2908 4795 50  0000 R CNN
+F 1 "4.7 uF" H 2908 4795 50  0000 R CNN
 F 2 "Capacitors_SMD:C_0603" H 3000 4750 50  0001 C CNN
 F 3 "~" H 3000 4750 50  0001 C CNN
@@
 P 5500 3150
 F 0 "C201" H 5408 3104 50  0000 R CNN
-F 1 "2.2 uF" H 5408 3195 50  0000 R CNN
+F 1 "4.7 uF" H 5408 3195 50  0000 R CNN
 F 2 "Capacitors_SMD:C_0603" H 5500 3150 50  0001 C CNN
 F 3 "~" H 5500 3150 50  0001 C CNN
@@
 P 5700 2800
 F 0 "R203" H 5759 2846 50  0000 L CNN
-F 1 "TBD" H 5759 2755 50  0000 L CNN
+F 1 "DNI" H 5759 2755 50  0000 L CNN
 F 2 "Resistors_SMD:R_0402" H 5700 2800 50  0001 C CNN
 F 3 "~" H 5700 2800 50  0001 C CNN
@@
 P 5700 2200
 F 0 "C202" H 5608 2154 50  0000 R CNN
-F 1 "2.2 uF" H 5608 2245 50  0000 R CNN
+F 1 "4.7 uF" H 5608 2245 50  0000 R CNN
 F 2 "Capacitors_SMD:C_0603" H 5700 2200 50  0001 C CNN
 F 3 "~" H 5700 2200 50  0001 C CNN
@@
 P 6000 2650
 F 0 "R205" V 5804 2650 50  0000 C CNN
-F 1 "TBD" V 5895 2650 50  0000 C CNN
+F 1 "DNI" V 5895 2650 50  0000 C CNN
 F 2 "Resistors_SMD:R_0402" H 6000 2650 50  0001 C CNN
 F 3 "~" H 6000 2650 50  0001 C CNN
@@
 Text Notes 12050 1000 0    50   ~ 0
 Murata JSC connector looks nice, but hard to source...
+Text Notes 4800 6800 0    50   ~ 0
+VOUT+ = 1.2 V × (R1 + R2) / R2\nVOUT- = –1.22 V × (R3 + R4) / R4\nR must be no less than 50k
+Text Notes 4850 5300 0    50   ~ 0
+R1
+Text Notes 4850 5600 0    50   ~ 0
+R2
+Text Notes 4850 5900 0    50   ~ 0
+R4
+Text Notes 4850 6200 0    50   ~ 0
+R3
 $EndSCHEMATC
