File: hardware/output_driver.sch (KiCad schematic (older format))
At the start: 12 parts

Commit message: more work on tdr schematic
Parts:
- U?: symbol synth_lib:ADCMP580 -> tdr-rescue:ADCMP580-synth_lib
Changed lines of the file:
@@
 $EndDescr
 $Comp
-L synth_lib:ADCMP580 U?
+L tdr-rescue:ADCMP580-synth_lib U?
 U 1 1 5BC2B59B
 P 5700 3350

Commit message: work on tdr schematic..
Parts:
- U?: symbol tdr-rescue:ADCMP580-synth_lib -> tdr-rescue:ADCMP580-synth_lib-tdr-rescue
Changed lines of the file:
@@
 $Descr A4 11693 8268
 encoding utf-8
-Sheet 5 9
+Sheet 5 8
 Title ""
 Date ""
@@
 $EndDescr
 $Comp
-L tdr-rescue:ADCMP580-synth_lib U?
+L tdr-rescue:ADCMP580-synth_lib-tdr-rescue U?
 U 1 1 5BC2B59B
 P 5700 3350

Commit message: footprint assignment
Parts:
- C501, C502, C503, C504: renamed from C?; footprint (none) -> Capacitors_SMD:C_0402
- R501, R502, R503, R504, R505, R506, R507: renamed from R?; footprint (none) -> Resistors_SMD:R_0402
- U501: renamed from U?; footprint (none) -> Housings_DFN_QFN:QFN-16-1EP_3x3mm_Pitch0.5mm

Commit message: layout of low speed digital traces
Parts:
- R506, R507: footprint Resistors_SMD:R_0402 -> Resistors_SMD:R_0201
Changed lines of the file:
@@
 F 0 "R507" V 8000 3450 50  0000 L CNN
 F 1 "JMP" V 8000 3250 50  0000 L CNN
-F 2 "Resistors_SMD:R_0402" H 8100 3400 50  0001 C CNN
+F 2 "Resistors_SMD:R_0201" H 8100 3400 50  0001 C CNN
 F 3 "~" H 8100 3400 50  0001 C CNN
 	1    8100 3400
@@
 F 0 "R506" V 8000 3350 50  0000 L CNN
 F 1 "JMP" V 8000 3150 50  0000 L CNN
-F 2 "Resistors_SMD:R_0402" H 8100 3300 50  0001 C CNN
+F 2 "Resistors_SMD:R_0201" H 8100 3300 50  0001 C CNN
 F 3 "~" H 8100 3300 50  0001 C CNN
 	1    8100 3300

Commit message: fixed CML termination.. ready to order?
Parts:
- removed R501: 50, Resistors_SMD:R_0402, symbol Device:R_Small
- C501, C502, C503, C504: value .01 uF -> 10 nF
Connections:
- net +3V3: now reaches C501.1, U501.1 (Vtp), U501.4 (Vtn)
Other:
- moved on the sheet: C501
Changed lines of the file:
@@
 AR Path="/5BC2B41E/5BC2B5D0" Ref="C502"  Part="1"
 F 0 "C502" H 4850 2450 50  0000 L CNN
-F 1 ".01 uF" H 4850 2350 50  0000 L CNN
+F 1 "10 nF" H 4850 2350 50  0000 L CNN
 F 2 "Capacitors_SMD:C_0402" H 5250 2400 50  0001 C CNN
 F 3 "~" H 5250 2400 50  0001 C CNN
@@
 AR Path="/5BC2B41E/5BC2B5EB" Ref="C503"  Part="1"
 F 0 "C503" H 5392 4296 50  0000 L CNN
-F 1 ".01 uF" H 5392 4205 50  0000 L CNN
+F 1 "10 nF" H 5392 4205 50  0000 L CNN
 F 2 "Capacitors_SMD:C_0402" H 5300 4250 50  0001 C CNN
 F 3 "~" H 5300 4250 50  0001 C CNN
@@
 AR Path="/5BC2B41E/5BC2B60C" Ref="C504"  Part="1"
 F 0 "C504" H 6192 2446 50  0000 L CNN
-F 1 ".01 uF" H 6192 2355 50  0000 L CNN
+F 1 "10 nF" H 6192 2355 50  0000 L CNN
 F 2 "Capacitors_SMD:C_0402" H 6100 2400 50  0001 C CNN
 F 3 "~" H 6100 2400 50  0001 C CNN
@@
 Wire Wire Line
 	5650 2650 5650 2700
-Wire Wire Line
-	4950 3500 5050 3500
-Wire Wire Line
-	4950 3200 5050 3200
 Wire Wire Line
 	5650 4000 5650 4900
@@
 CLK_IN_N
 $Comp
-L Device:R_Small R?
-U 1 1 5BC32D77
-P 4850 3800
-AR Path="/5BC41CC8/5BC32D77" Ref="R?"  Part="1"
-AR Path="/5BC2B41E/5BC32D77" Ref="R501"  Part="1"
-F 0 "R501" V 4750 3850 50  0000 L CNN
-F 1 "50" V 4750 3650 50  0000 L CNN
-F 2 "Resistors_SMD:R_0402" H 4850 3800 50  0001 C CNN
-F 3 "~" H 4850 3800 50  0001 C CNN
-	1    4850 3800
-	-1   0    0    1
-$EndComp
-Wire Wire Line
-	4950 3200 4950 3500
-Connection ~ 4950 3500
-$Comp
-L power:GND #PWR?
-U 1 1 5BC33DFF
-P 4850 3950
-AR Path="/5BC41CC8/5BC33DFF" Ref="#PWR?"  Part="1"
-AR Path="/5BC2B41E/5BC33DFF" Ref="#PWR0245"  Part="1"
-F 0 "#PWR0245" H 4850 3700 50  0001 C CNN
-F 1 "GND" V 4900 3950 50  0001 C CNN
-F 2 "" H 4850 3950 50  0001 C CNN
-F 3 "" H 4850 3950 50  0001 C CNN
-	1    4850 3950
-	1    0    0    -1
-$EndComp
-Wire Wire Line
-	4850 3500 4850 3700
-Wire Wire Line
-	4850 3900 4850 3950
-$Comp
 L Device:C_Small C?
 U 1 1 5BC34BA3
-P 4450 3800
+P 4500 4000
 AR Path="/5BC41CC8/5BC34BA3" Ref="C?"  Part="1"
 AR Path="/5BC2B41E/5BC34BA3" Ref="C501"  Part="1"
-F 0 "C501" H 4542 3846 50  0000 L CNN
-F 1 ".01 uF" H 4542 3755 50  0000 L CNN
-F 2 "Capacitors_SMD:C_0402" H 4450 3800 50  0001 C CNN
-F 3 "~" H 4450 3800 50  0001 C CNN
-	1    4450 3800
-	1    0    0    -1
-$EndComp
-Wire Wire Line
-	4450 3500 4450 3700
+F 0 "C501" H 4592 4046 50  0000 L CNN
+F 1 "10 nF" H 4592 3955 50  0000 L CNN
+F 2 "Capacitors_SMD:C_0402" H 4500 4000 50  0001 C CNN
+F 3 "~" H 4500 4000 50  0001 C CNN
+	1    4500 4000
+	1    0    0    -1
+$EndComp
 $Comp
 L power:GND #PWR?
 U 1 1 5BC35338
-P 4450 3950
+P 4500 4150
 AR Path="/5BC41CC8/5BC35338" Ref="#PWR?"  Part="1"
 AR Path="/5BC2B41E/5BC35338" Ref="#PWR0246"  Part="1"
-F 0 "#PWR0246" H 4450 3700 50  0001 C CNN
-F 1 "GND" V 4500 3950 50  0001 C CNN
-F 2 "" H 4450 3950 50  0001 C CNN
-F 3 "" H 4450 3950 50  0001 C CNN
-	1    4450 3950
-	1    0    0    -1
-$EndComp
-Wire Wire Line
-	4450 3950 4450 3900
+F 0 "#PWR0246" H 4500 3900 50  0001 C CNN
+F 1 "GND" V 4550 4150 50  0001 C CNN
+F 2 "" H 4500 4150 50  0001 C CNN
+F 3 "" H 4500 4150 50  0001 C CNN
+	1    4500 4150
+	1    0    0    -1
+$EndComp
+Wire Wire Line
+	4500 4150 4500 4100
 Wire Wire Line
 	4000 3300 5050 3300
 Wire Wire Line
 	4000 3400 5050 3400
-Wire Wire Line
-	4450 3500 4850 3500
-Connection ~ 4850 3500
-Wire Wire Line
-	4850 3500 4950 3500
+$Comp
+L power:+3V3 #PWR0248
+U 1 1 5C348861
+P 5000 3500
+F 0 "#PWR0248" H 5000 3350 50  0001 C CNN
+F 1 "+3V3" V 5015 3628 50  0000 L CNN
+F 2 "" H 5000 3500 50  0001 C CNN
+F 3 "" H 5000 3500 50  0001 C CNN
+	1    5000 3500
+	0    -1   -1   0
+$EndComp
+Wire Wire Line
+	5000 3500 5050 3500
+$Comp
+L power:+3V3 #PWR0249
+U 1 1 5C348FB2
+P 5000 3200
+F 0 "#PWR0249" H 5000 3050 50  0001 C CNN
+F 1 "+3V3" V 5015 3328 50  0000 L CNN
+F 2 "" H 5000 3200 50  0001 C CNN
+F 3 "" H 5000 3200 50  0001 C CNN
+	1    5000 3200
+	0    -1   -1   0
+$EndComp
+Wire Wire Line
+	5050 3200 5000 3200
+$Comp
+L power:+3V3 #PWR0253
+U 1 1 5C349D6E
+P 4500 3800
+F 0 "#PWR0253" H 4500 3650 50  0001 C CNN
+F 1 "+3V3" H 4515 3973 50  0000 C CNN
+F 2 "" H 4500 3800 50  0001 C CNN
+F 3 "" H 4500 3800 50  0001 C CNN
+	1    4500 3800
+	1    0    0    -1
+$EndComp
+Wire Wire Line
+	4500 3800 4500 3900
 $EndSCHEMATC

Commit message: schematic cleanup, BOM consolidation
Parts:
- R503: value TBD -> 1k
Changed lines of the file:
@@
 AR Path="/5BC2B41E/5BC2B5FC" Ref="R503"  Part="1"
 F 0 "R503" V 5650 2400 50  0000 L CNN
-F 1 "TBD" V 5650 2200 50  0000 L CNN
+F 1 "1k" V 5650 2200 50  0000 L CNN
 F 2 "Resistors_SMD:R_0402" H 5750 2350 50  0001 C CNN
 F 3 "~" H 5750 2350 50  0001 C CNN
