File: hardware/tdr.kicad_pcb (KiCad board)
At the start: 4 copper layers, 101 x 47 mm, 240 parts, among them J201 Conn_02x01, J202 Conn_Coaxial, J203 Conn_Coaxial, J204 Conn_Coaxial, J205 Conn_Coaxial, J207 Conn_Coaxial, J208 Conn_Coaxial, J209 Conn_Coaxial, J210 Barrel_Jack_Switch, J801 Conn_02x06_Counter_Clockwise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

Commit message: clean up of interactive BOM page, waiting on PCBs
Parts:
- C201, C202, C205, C212, C213, C322, C324, C325, C406, C601: value 2.2 uF -> 4.7 uF
- C211: value 2.2 uF -> 10 uF
- C705, C706: value TBD -> 10 pF
- C707, C708: value 1 uF -> 4.7 uF
- C802, C806: value 1 uF -> DNP
- R203, R205: value TBD -> DNI
- R216, R219: value TBD -> 1M
- R217, R218: value TBD -> 332k
- R220, R221, R306, R702: value R_Small -> JMP
- R304, R403, R503: value TBD -> 1k
- U201: value LD39100 -> LD39100PU33R
Changed lines of the file:
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@@
       (effects (font (size 0.7 0.7) (thickness 0.15)))
     )
-    (fp_text value "2.2 uF" (at 0 1.9 90) (layer F.Fab)
+    (fp_text value "4.7 uF" (at 0 1.9 90) (layer F.Fab)
       (effects (font (size 0.7 0.7) (thickness 0.15)))
     )
@@
       (effects (font (size 0.7 0.7) (thickness 0.15)))
     )
-    (fp_text value "2.2 uF" (at 0 1.9 90) (layer F.Fab)
+    (fp_text value "4.7 uF" (at 0 1.9 90) (layer F.Fab)
       (effects (font (size 0.7 0.7) (thickness 0.15)))
     )
@@
       (effects (font (size 0.7 0.7) (thickness 0.15)))
     )
-    (fp_text value "2.2 uF" (at 0 1.9 180) (layer F.Fab)
+    (fp_text value "4.7 uF" (at 0 1.9 180) (layer F.Fab)
       (effects (font (size 0.7 0.7) (thickness 0.15)))
     )
@@
       (effects (font (size 0.7 0.7) (thickness 0.15)))
     )
-    (fp_text value "2.2 uF" (at 0 1.9 270) (layer F.Fab)
+    (fp_text value "10 uF" (at 0 1.9 270) (layer F.Fab)
       (effects (font (size 0.7 0.7) (thickness 0.15)))
     )
@@
       (effects (font (size 0.7 0.7) (thickness 0.15)))
     )
-    (fp_text value "2.2 uF" (at 0 1.9 180) (layer F.Fab)
+    (fp_text value "4.7 uF" (at 0 1.9 180) (layer F.Fab)
       (effects (font (size 0.7 0.7) (thickness 0.15)))
     )
@@
       (effects (font (size 0.7 0.7) (thickness 0.15)))
     )
-    (fp_text value "2.2 uF" (at 0 1.9 270) (layer F.Fab)
+    (fp_text value "4.7 uF" (at 0 1.9 270) (layer F.Fab)
       (effects (font (size 0.7 0.7) (thickness 0.15)))
     )
@@
       (effects (font (size 0.7 0.7) (thickness 0.15)))
     )
-    (fp_text value "2.2 uF" (at 0 1.9) (layer F.Fab)
+    (fp_text value "4.7 uF" (at 0 1.9) (layer F.Fab)
       (effects (font (size 0.7 0.7) (thickness 0.15)))
     )
@@
       (effects (font (size 0.7 0.7) (thickness 0.15)))
     )
-    (fp_text value "2.2 uF" (at 0 1.9 180) (layer F.Fab)
+    (fp_text value "4.7 uF" (at 0 1.9 180) (layer F.Fab)
       (effects (font (size 0.7 0.7) (thickness 0.15)))
     )
@@
       (effects (font (size 0.7 0.7) (thickness 0.15)))
     )
-    (fp_text value "2.2 uF" (at 0 1.9 180) (layer F.Fab)
+    (fp_text value "4.7 uF" (at 0 1.9 180) (layer F.Fab)
       (effects (font (size 0.7 0.7) (thickness 0.15)))
     )
@@
       (effects (font (size 0.7 0.7) (thickness 0.15)) (justify mirror))
     )
-    (fp_text value "2.2 uF" (at 0 -1.9) (layer B.Fab)
+    (fp_text value "4.7 uF" (at 0 -1.9) (layer B.Fab)
       (effects (font (size 0.7 0.7) (thickness 0.15)) (justify mirror))
     )
@@
       (effects (font (size 0.7 0.7) (thickness 0.15)))
     )
-    (fp_text value TBD (at 0 1.7) (layer F.Fab)
+    (fp_text value "10 pF" (at 0 1.7) (layer F.Fab)
       (effects (font (size 0.7 0.7) (thickness 0.15)))
     )
@@
       (effects (font (size 0.7 0.7) (thickness 0.15)))
     )
-    (fp_text value TBD (at 0 1.7) (layer F.Fab)
+    (fp_text value "10 pF" (at 0 1.7) (layer F.Fab)
       (effects (font (size 0.7 0.7) (thickness 0.15)))
     )
@@
       (effects (font (size 0.7 0.7) (thickness 0.15)))
     )
-    (fp_text value "1 uF" (at 0 1.9 270) (layer F.Fab)
+    (fp_text value "4.7 uF" (at 0 1.9 270) (layer F.Fab)
       (effects (font (size 0.7 0.7) (thickness 0.15)))
     )
@@
       (effects (font (size 0.7 0.7) (thickness 0.15)))
     )
-    (fp_text value "1 uF" (at 0 1.9) (layer F.Fab)
+    (fp_text value "4.7 uF" (at 0 1.9) (layer F.Fab)
       (effects (font (size 0.7 0.7) (thickness 0.15)))
     )
@@
       (effects (font (size 0.7 0.7) (thickness 0.15)))
     )
-    (fp_text value "1 uF" (at 0 1.9 180) (layer F.Fab)
+    (fp_text value DNP (at 0 1.9 180) (layer F.Fab)
       (effects (font (size 0.7 0.7) (thickness 0.15)))
     )
@@
       (effects (font (size 0.7 0.7) (thickness 0.15)))
     )
-    (fp_text value "1 uF" (at 0 1.9) (layer F.Fab)
+    (fp_text value DNP (at 0 1.9) (layer F.Fab)
       (effects (font (size 0.7 0.7) (thickness 0.15)))
     )
@@
       (effects (font (size 0.7 0.7) (thickness 0.15)))
     )
-    (fp_text value TBD (at 0 1.8) (layer F.Fab)
+    (fp_text value DNI (at 0 1.8) (layer F.Fab)
       (effects (font (size 0.7 0.7) (thickness 0.15)))
     )
@@
       (effects (font (size 0.7 0.7) (thickness 0.15)))
     )
-    (fp_text value TBD (at 0 1.8 270) (layer F.Fab)
+    (fp_text value DNI (at 0 1.8 270) (layer F.Fab)
       (effects (font (size 0.7 0.7) (thickness 0.15)))
     )
@@
       (effects (font (size 0.7 0.7) (thickness 0.15)))
     )
-    (fp_text value TBD (at 0 1.8 180) (layer F.Fab)
+    (fp_text value 1M (at 0 1.8 180) (layer F.Fab)
       (effects (font (size 0.7 0.7) (thickness 0.15)))
     )
@@
       (effects (font (size 0.7 0.7) (thickness 0.15)))
     )
-    (fp_text value TBD (at 0 1.8) (layer F.Fab)
+    (fp_text value 332k (at 0 1.8) (layer F.Fab)
       (effects (font (size 0.7 0.7) (thickness 0.15)))
     )
@@
       (effects (font (size 0.7 0.7) (thickness 0.15)))
     )
-    (fp_text value TBD (at 0 1.8 90) (layer F.Fab)
+    (fp_text value 332k (at 0 1.8 90) (layer F.Fab)
       (effects (font (size 0.7 0.7) (thickness 0.15)))
     )
@@
       (effects (font (size 0.7 0.7) (thickness 0.15)))
     )
-    (fp_text value TBD (at 0 1.8 270) (layer F.Fab)
+    (fp_text value 1M (at 0 1.8 270) (layer F.Fab)
       (effects (font (size 0.7 0.7) (thickness 0.15)))
     )
@@
       (effects (font (size 0.7 0.7) (thickness 0.15)))
     )
-    (fp_text value R_Small (at 0 1.8 90) (layer F.Fab)
+    (fp_text value JMP (at 0 1.8 90) (layer F.Fab)
       (effects (font (size 0.7 0.7) (thickness 0.15)))
     )
@@
       (effects (font (size 0.7 0.7) (thickness 0.15)))
     )
-    (fp_text value R_Small (at 0 1.8) (layer F.Fab)
+    (fp_text value JMP (at 0 1.8) (layer F.Fab)
       (effects (font (size 0.7 0.7) (thickness 0.15)))
     )
@@
       (effects (font (size 0.7 0.7) (thickness 0.15)))
     )
-    (fp_text value TBD (at 0 1.8 90) (layer F.Fab)
+    (fp_text value 1k (at 0 1.8 90) (layer F.Fab)
       (effects (font (size 0.7 0.7) (thickness 0.15)))
     )
@@
       (effects (font (size 0.7 0.7) (thickness 0.15)))
     )
-    (fp_text value R_Small (at 0 1.8) (layer F.Fab)
+    (fp_text value JMP (at 0 1.8) (layer F.Fab)
       (effects (font (size 0.7 0.7) (thickness 0.15)))
     )
@@
       (effects (font (size 0.7 0.7) (thickness 0.15)))
     )
-    (fp_text value TBD (at 0 1.8 90) (layer F.Fab)
+    (fp_text value 1k (at 0 1.8 90) (layer F.Fab)
       (effects (font (size 0.7 0.7) (thickness 0.15)))
     )
@@
       (effects (font (size 0.7 0.7) (thickness 0.15)))
     )
-    (fp_text value TBD (at 0 1.8 270) (layer F.Fab)
+    (fp_text value 1k (at 0 1.8 270) (layer F.Fab)
       (effects (font (size 0.7 0.7) (thickness 0.15)))
     )
@@
       (effects (font (size 0.7 0.7) (thickness 0.15)))
     )
-    (fp_text value R_Small (at 0 1.8) (layer F.Fab)
+    (fp_text value JMP (at 0 1.8) (layer F.Fab)
       (effects (font (size 0.7 0.7) (thickness 0.15)))
     )
@@
       (effects (font (size 0.7 0.7) (thickness 0.15)))
     )
-    (fp_text value LD39100 (at 0 2.575 90) (layer F.Fab)
+    (fp_text value LD39100PU33R (at 0 2.575 90) (layer F.Fab)
       (effects (font (size 0.7 0.7) (thickness 0.15)))
     )
@@
       (effects (font (size 0.7 0.7) (thickness 0.15)) (justify mirror))
     )
-    (fp_text value "2.2 uF" (at 0 -1.9 180) (layer B.Fab)
+    (fp_text value "4.7 uF" (at 0 -1.9 180) (layer B.Fab)
       (effects (font (size 0.7 0.7) (thickness 0.15)) (justify mirror))
     )
